File: cpapboi.kicad_sch (KiCad schematic)
At the start: 11 parts, among them U1 STM32G0B1CBTx, U2 TPS54202DDC, U3 TPS54202DDC

Commit message: wip
Parts:
- added C10, C11, C12: 100nF, Capacitor_SMD:C_0603_1608Metric, symbol Device:C_Small
- added C13: 100pF, Capacitor_SMD:C_0603_1608Metric, symbol Device:C_Small
- added C14, C15: 22uF, Capacitor_SMD:C_0805_2012Metric, symbol Device:C_Small
- added C16, C17, C18: 10uF, Capacitor_SMD:C_0603_1608Metric, symbol Device:C_Small
- added F1: Fuse_Small, Fuse:Fuseholder_Littelfuse_Nano2_154x, symbol Device:Fuse_Small
- added J2, J3, J4: Screw Terminal, TerminalBlock_CUI:TerminalBlock_CUI_TB007-508-02_1x02_P5.08mm_Horizontal, symbol Connector:Conn_01x02_Socket
- added J5, J6: JST-XH, Connector_JST:JST_XH_S2B-XH-A_1x02_P2.50mm_Horizontal, symbol Connector:Conn_01x02_Pin
- added R10, R13: 100k, Resistor_SMD:R_0603_1608Metric, symbol Device:R_Small
- added R11: 13.3k, Resistor_SMD:R_0603_1608Metric, symbol Device:R_Small
- added R12, R9: 49.9, Resistor_SMD:R_0603_1608Metric, symbol Device:R_Small
- added R14: 5.23k, Resistor_SMD:R_0603_1608Metric, symbol Device:R_Small
- added U5: ME6211C33M5, Package_TO_SOT_SMD:SOT-23-5, symbol Regulator_Linear:ME6211C33M5
- added U6: SN65HVD231, Package_SO:SOIC-8_3.9x4.9mm_P1.27mm, symbol Interface_CAN_LIN:SN65HVD231
- C6: value 100pF -> 10uF; footprint Capacitor_SMD:C_0603_1608Metric -> Capacitor_SMD:C_1206_3216Metric
Connections:
- net +24V: now reaches C6.1
- net +24V: now also C1.1, C2.1, U2.3 (VIN), U3.3 (VIN), C11.1, F1.2
- net GND: now reaches C6.2
- net GND: now also C1.2, C2.2, C3.2, C4.2, U2.1 (GND), U3.1 (GND), C11.2, C14.2, C15.2, C16.2, C17.2, C18.2, R11.1, R14.1, U5.2 (V_{SS})
- net at L2.1: now also U3.2 (SW), C12.2
- net +12V: now reaches L2.2
- net +12V: now also C14.1, C15.1, R12.2
- net at C5.1: now also R10.1, R9.1
- net at C5.2: now also U2.4 (FB), R10.2, R11.2
- net at L1.1: now also U2.2 (SW), C10.2
- net +5V: now reaches L1.2
- net +5V: now also C3.1, C4.1, C16.1, R9.2, U5.1 (V_{IN}), U5.3 (CE)
- net at U2.6 (BOOT): now also C10.1
- net at U3.4 (FB): now also C13.2, R13.2, R14.2
- net at U3.6 (BOOT): now also C12.1
- new net: C13.1, R12.1, R13.1
- new net +24V_IN: F1.1
- new net +3.3V: C17.1, C18.1, U5.5 (V_{OUT})
- no-connect marks 0 -> 2
Other:
- added sheet Filament Sensor (filament_sensor.kicad_sch)
- added sheet WS7040 Control (ws7040.kicad_sch)
- moved on the sheet: C1, C2, C3, C4, C5, L1, L2, U1, U2

Commit message: stuff
Parts:
- added J7: Conn_ARM_SWD_TagConnect_TC2030, Connector:Tag-Connect_TC2030-IDC-FP_2x03_P1.27mm_Vertical, symbol Connector:Conn_ARM_SWD_TagConnect_TC2030
Changed lines of the file:
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@@
+	)
+	(symbol
+		(lib_id "Connector:Conn_ARM_SWD_TagConnect_TC2030")
+		(at 180.34 55.88 0)
+		(unit 1)
+		(body_style 1)
+		(exclude_from_sim no)
+		(in_bom no)
+		(on_board yes)
+		(in_pos_files yes)
+		(dnp no)
+		(fields_autoplaced yes)
+		(property "Reference" "J7"
+			(at 173.99 54.61 0)
+			(show_name no)
+			(do_not_autoplace no)
+			(effects
+				(font
+					(size 1.27 1.27)
+				)
+				(justify right)
+			)
+		)
+		(property "Value" "Conn_ARM_SWD_TagConnect_TC2030"
+			(at 173.99 57.15 0)
+			(show_name no)
+			(do_not_autoplace no)
+			(effects
+				(font
+					(size 1.27 1.27)
+				)
+				(justify right)
+			)
+		)
+		(property "Footprint" "Connector:Tag-Connect_TC2030-IDC-FP_2x03_P1.27mm_Vertical"
+			(at 180.34 73.66 0)
+			(hide yes)
+			(show_name no)
+			(do_not_autoplace no)
+			(effects
+				(font
+					(size 1.27 1.27)
+				)
+			)
+		)
+		(property "Datasheet" "https://www.tag-connect.com/wp-content/uploads/bsk-pdf-manager/TC2030-CTX_1.pdf"
+			(at 180.34 71.12 0)
+			(hide yes)
+			(show_name no)
+			(do_not_autoplace no)
+			(effects
+				(font
+					(size 1.27 1.27)
+				)
+			)
+		)
+		(property "Description" "Tag-Connect ARM Cortex SWD JTAG connector, 6 pin"
+			(at 180.34 55.88 0)
+			(hide yes)
+			(show_name no)
+			(do_not_autoplace no)
+			(effects
+				(font
+					(size 1.27 1.27)
+				)
+			)
+		)
+		(pin "4"
+		)
+		(pin "3"
+		)
+		(pin "6"
+		)
+		(pin "5"
+		)
+		(pin "1"
+		)
+		(pin "2"
+		)
+		(instances
+			(project "cpapboi"
+				(path "/320a9d09-725c-47b2-ba01-b8bc02b3665e"
+					(reference "J7")
+					(unit 1)
+				)
+			)
+		)
 	)
 	(symbol

Commit message: wip
Parts:
- added D1: SP0505BAJT, Package_TO_SOT_SMD:SOT-363_SC-70-6, symbol Power_Protection:SP0505BAJT
- added J8: USB_C_Receptacle_USB2.0_16P, Connector_USB:USB_C_Receptacle_XKB_U262-16XN-4BVC11, symbol Connector:USB_C_Receptacle_USB2.0_16P
- added R16: 49.9, Resistor_SMD:R_0603_1608Metric, symbol Device:R_Small
- added R17, R18: 5.1k, Resistor_SMD:R_0603_1608Metric, symbol Device:R_Small
- added R19: 100k, Resistor_SMD:R_0603_1608Metric, symbol Device:R_Small
- added R20: 56k, Resistor_SMD:R_0603_1608Metric, symbol Device:R_Small
- added U7: TPS2116DRL, Package_TO_SOT_SMD:SOT-583-8, symbol Power_Management:TPS2116DRL
Connections:
- net +24V_IN: now also J2.1 (Pin_1), J3.1 (Pin_1), J4.1 (Pin_1)
- net +5V: now also R19.2, U7.3 (VIN1), U7.5 (MODE); no longer C16.1, U5.1 (V_{IN}), U5.3 (CE)
- net GND: now also J2.2 (Pin_2), J3.2 (Pin_2), J4.2 (Pin_2), D1.2 (A), J8.A1 (GND), J8.A12 (GND), J8.B1 (GND), J8.B12 (GND), J8.SH (SHIELD), R17.1, R18.1, R20.1, U7.1 (GND)
- net D-: now reaches U1.33 (PA9/PA11)
- net D-: now also D1.4 (K), J8.A7 (D-), J8.B7 (D-)
- net D+: now reaches U1.34 (PA10/PA12)
- net D+: now also D1.3 (K), J8.A6 (D+), J8.B6 (D+)
- net SWDIO: now reaches U1.35 (PA13)
- net SWCLK: now reaches U1.36 (PA14)
- net CAN_RX: now reaches U1.47 (PB8)
- net CAN_TX: now reaches U1.48 (PB9)
- new net: C16.1, U5.1 (V_{IN}), U5.3 (CE), U7.2 (VOUT), U7.7 (VOUT)
- new net: R19.1, R20.2, U7.4 (PR1)
- new net: J8.A5 (CC1), R17.2
- new net: J8.B5 (CC2), R18.2
- new net VBUS: D1.1 (K), J8.A4 (VBUS), J8.A9 (VBUS), J8.B4 (VBUS), J8.B9 (VBUS), U7.6 (VIN2)
- no-connect marks 2 -> 5
Other:
- moved on the sheet: C16, C17, C18, J2, J3, J4, J5, J6, U5, U6

Commit message: wip
Parts:
- added C20, C21: 12pF, Capacitor_SMD:C_0603_1608Metric, symbol Device:C_Small
- added C22, C23, C24, C26: 100nF, Capacitor_SMD:C_0603_1608Metric, symbol Device:C_Small
- added C25: 10uF, Capacitor_SMD:C_0603_1608Metric, symbol Device:C_Small
- added R21, R22: 10k, Resistor_SMD:R_0603_1608Metric, symbol Device:R_Small
- added SW1, SW2: SW_MEC_5E, symbol Switch:SW_MEC_5E
- added Y1: 25MHz, Crystal:Crystal_SMD_3225-4Pin_3.2x2.5mm, symbol Device:Crystal_GND24_Small
Connections:
- net SWCLK is gone; now on net SWCLK/BOOT0: U1.36 (PA14)
- net +3.3V: now also J7.1 (VCC), U1.4 (VBAT), U1.5 (VREF+), U1.6 (VDD), C22.1, C23.1, C24.1, C25.1, R22.1, SW2.1, SW2.2
- net GND: now also J7.5 (GND), U1.7 (VSS), C20.2, C21.2, C22.2, C23.2, C24.2, C25.2, C26.2, R21.2, SW1.1, SW1.2
- net SWDIO: now also J7.2 (SWDIO)
- net NRST: now reaches J7.3 (~{RESET})
- net NRST: now also U1.10 (PF2), C26.1, R22.2, SW1.3 (K), SW1.4 (A)
- net SWCLK/BOOT0: now reaches J7.4 (SWCLK)
- net SWCLK/BOOT0: now also R21.1, SW2.3 (K), SW2.4 (A)
- net at U1.8 (PF0): now also C20.1, Y1.1
- net at U1.9 (PF1): now also C21.1, Y1.3
- new net: Y1.2 (G), Y1.4 (G)
- no-connect marks 5 -> 6
Other:
- moved on the sheet: J7
